Commit message: bug in kinematics

File: packages/manipulator/urdf/arm.urdf (robot description, URDF)
Before this commit: robot arm, 17 links, 16 joints
Joints:
- removed joint basetomotor0
- added joint base0tomotor: type fixed, parent joint0base, child joint0motor, origin xyz=0 0 -0.05715 rpy=0 0 0

Commit message: Post CIRC init

File: packages/manipulator/urdf/arm.urdf (robot description, URDF)
Before this commit: robot arm, 17 links, 16 joints
Joints:
- joint base0tomotor: origin xyz=0 0 -0.05715 rpy=0 0 0 -> xyz=0 0 -0.5715 rpy=0 0 0
- joint basetomotor4: origin xyz=-0.001778 0.02667 0.030734  rpy=-1.5708 0 0 -> xyz=-0.001778 0.02667 0.030734  rpy=0 1.5708 0
- joint placement: origin xyz=0 0 0.480 rpy=0 0 0 -> xyz=0 0 0.450 rpy=0 0 0
- joint tiprotary: type continuous -> fixed
